Commit message: Added mesh to this package

File: mantaray_transforms/urdf/mantaray_robot.xacro (robot description, xacro)
@@ -1,5 +1,5 @@
 <?xml version="1.0"?>
 <robot xmlns:xacro="http://www.ros.org/wiki/xacro" name="mantaray">
-  <xacro:property name="description_pkg" value="mantaray_description" />
+  <xacro:property name="description_pkg" value="mantaray_transforms" />
   <!-- Base Link -->
   <link name="base_link">

Commit message: Finished creating urdf mimicking their transforms

File: mantaray_transforms/urdf/mantaray_robot.xacro (robot description, xacro)
@@ -1,4 +1,7 @@
 <?xml version="1.0"?>
 <robot xmlns:xacro="http://www.ros.org/wiki/xacro" name="mantaray">
+  <material name="green">
+    <color rgba="0.1 0.8 0.1 0.8"/>
+  </material>
   <xacro:property name="description_pkg" value="mantaray_transforms" />
   <!-- Base Link -->
@@ -6,6 +9,7 @@
     <visual>
       <geometry>
-        <mesh filename="$(find ${description_pkg})/meshes/visual_base_link.stl"/>
+        <mesh filename="package://mantaray_transforms/meshes/visual_base_link.stl"/>
       </geometry>
+      <material name="green"/>
     </visual>
     <collision>
@@ -31,5 +35,5 @@
     <parent link="base_link"/>
     <child link="imu_link"/>
-    <origin xyz="0.013 0.005 0.01" rpy="0 0 0"/> <!-- Adjust position inside hull -->
+    <origin xyz="0.05 -0.13 0.03" rpy="0 0 0"/> <!-- Adjust position inside hull -->
   </joint>
   <!-- DVL Sensor -->
@@ -49,5 +53,5 @@
     <parent link="base_link"/>
     <child link="dvl_link"/>
-    <origin xyz="0 0.04 0" rpy="0 0 0"/> <!-- Adjust position to right side -->
+    <origin xyz="-0.1 0 -0.13" rpy="0 0 0"/> <!-- Adjust position to right side -->
   </joint>
   <!-- Pressure Sensor -->
@@ -55,10 +59,10 @@
     <visual>
       <geometry>
-        <box size="0.05 0.05 0.05"/> <!-- Adjust size as needed -->
+        <box size="0.02 0.02 0.05"/> <!-- Adjust size as needed -->
       </geometry>
     </visual>
     <collision>
       <geometry>
-        <box size="0.05 0.05 0.05"/> <!-- Match visual size -->
+        <box size="0.02 0.02 0.05"/> <!-- Match visual size -->
       </geometry>
     </collision>
@@ -67,5 +71,5 @@
     <parent link="base_link"/>
     <child link="pressure_sensor_link"/>
-    <origin xyz="0 0 0" rpy="0 0 0"/> <!-- Adjust position underneath -->
+    <origin xyz="0 0 -0.13" rpy="0 0 0"/> <!-- Adjust position underneath -->
   </joint>
 </robot>

Commit message: Got transforms working and positioned the sensors accurately.

File: mantaray_transforms/urdf/mantaray_robot.xacro (robot description, xacro)
@@ -6,5 +6,5 @@
   <xacro:property name="description_pkg" value="mantaray_transforms" />
   <!-- Base Link -->
-  <link name="base_link">
+  <link name="mantaray/base_link">
     <visual>
       <geometry>
@@ -20,5 +20,5 @@
   </link>
   <!-- IMU Sensor -->
-  <link name="imu_link">
+  <link name="mantaray/imu_link">
     <visual>
       <geometry>
@@ -33,10 +33,10 @@
   </link>
   <joint name="imu_joint" type="fixed">
-    <parent link="base_link"/>
-    <child link="imu_link"/>
+    <parent link="mantaray/base_link"/>
+    <child link="mantaray/imu_link"/>
     <origin xyz="0.05 -0.13 0.03" rpy="0 0 0"/> <!-- Adjust position inside hull -->
   </joint>
   <!-- DVL Sensor -->
-  <link name="dvl_link">
+  <link name="mantaray/dvl_link">
     <visual>
       <geometry>
@@ -51,10 +51,10 @@
   </link>
   <joint name="dvl_joint" type="fixed">
-    <parent link="base_link"/>
-    <child link="dvl_link"/>
+    <parent link="mantaray/base_link"/>
+    <child link="mantaray/dvl_link"/>
     <origin xyz="-0.1 0 -0.13" rpy="0 0 0"/> <!-- Adjust position to right side -->
   </joint>
   <!-- Pressure Sensor -->
-  <link name="pressure_sensor_link">
+  <link name="mantaray/pressure_sensor_link">
     <visual>
       <geometry>
@@ -69,6 +69,6 @@
   </link>
   <joint name="pressure_sensor_joint" type="fixed">
-    <parent link="base_link"/>
-    <child link="pressure_sensor_link"/>
+    <parent link="mantaray/base_link"/>
+    <child link="mantaray/pressure_sensor_link"/>
     <origin xyz="0 0 -0.13" rpy="0 0 0"/> <!-- Adjust position underneath -->
   </joint>
